File: kicad/MySensors328p.kicad_pcb (KiCad board)
At the start: 2 copper layers, 27 x 18 mm, 22 parts, among them J1 U.FL, J2 U.FL, P1 HEADER_2x7, P2 HEADER_2x7, U1 NRF24L01, U3 ATmega328P-AU, Y1 16 MHz

Commit message: Add files via upload
Other:
- board text added: "ADC6"
- board text added: "ADC7"
- board text added: "AERF"
- board text added: "GND"
- board text added: "PB0"
- board text added: "PB1 /CE"
- board text added: "PB2/CSN"
- board text added: "PB3/ MOSI"
- board text added: "PB4/MISO"
- board text added: "PB5/SCK"
- board text added: "PB6"
- board text added: "PB7"
- board text added: "PC0"
- board text added: "PC1"
- board text added: "PC2"
- board text added: "PC3"
- board text added: "PC4"
- board text added: "PC5"
- board text added: "PC6"
- board text added: "PD0"
- board text added: "PD1"
- board text added: "PD2/ IRQ"
- board text added: "PD3/ RES"
- board text added: "PD4"
- board text added: "PD5"
- board text added: "PD6"
- board text added: "PD7"
- board text added: "VCC"
Changed lines of the file:
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@@
   (general
     (thickness 1.6)
-    (drawings 4)
+    (drawings 32)
     (tracks 408)
     (zones 0)
@@
     (31 B.Cu signal)
     (32 B.Adhes user)
-    (33 F.Adhes user hide)
-    (34 B.Paste user hide)
-    (35 F.Paste user hide)
+    (33 F.Adhes user)
+    (34 B.Paste user)
+    (35 F.Paste user)
     (36 B.SilkS user)
     (37 F.SilkS user)
-    (38 B.Mask user hide)
-    (39 F.Mask user hide)
+    (38 B.Mask user)
+    (39 F.Mask user)
     (40 Dwgs.User user)
     (41 Cmts.User user)
@@
     (46 B.CrtYd user hide)
     (47 F.CrtYd user)
-    (48 B.Fab user hide)
+    (48 B.Fab user)
     (49 F.Fab user hide)
   )
@@
     (tags "Surface mounted pin header SMD 2x07 2.54mm double row")
     (attr smd)
-    (fp_text reference P1 (at 5.015 0.05 90) (layer B.SilkS)
+    (fp_text reference P1 (at 5.015 2.85 90) (layer B.SilkS)
       (effects (font (size 1 1) (thickness 0.15)) (justify mirror))
     )
@@
     (tags "Surface mounted pin header SMD 2x07 2.54mm double row")
     (attr smd)
-    (fp_text reference P2 (at 4.875 0.005 90) (layer B.SilkS)
+    (fp_text reference P2 (at 4.825 3.005 90) (layer B.SilkS)
       (effects (font (size 1 1) (thickness 0.15)) (justify mirror))
     )
@@
     )
   )
+  (gr_text PC0 (at 137.5 91.55 180) (layer B.SilkS)
+    (effects (font (size 0.5 0.5) (thickness 0.1)) (justify mirror))
+  )
+  (gr_text PC2 (at 130.25 91.55 180) (layer B.SilkS)
+    (effects (font (size 0.5 0.5) (thickness 0.1)) (justify mirror))
+  )
+  (gr_text ADC7 (at 137.75 94 180) (layer B.SilkS)
+    (effects (font (size 0.5 0.5) (thickness 0.1)) (justify mirror))
+  )
+  (gr_text PC3 (at 130.2 94 180) (layer B.SilkS)
+    (effects (font (size 0.5 0.5) (thickness 0.1)) (justify mirror))
+  )
+  (gr_text PC1 (at 137.6 96.55 180) (layer B.SilkS)
+    (effects (font (size 0.5 0.5) (thickness 0.1)) (justify mirror))
+  )
+  (gr_text PC4 (at 130.2 96.6 180) (layer B.SilkS)
+    (effects (font (size 0.5 0.5) (thickness 0.1)) (justify mirror))
+  )
+  (gr_text PC5 (at 137.55 99.1 180) (layer B.SilkS)
+    (effects (font (size 0.5 0.5) (thickness 0.1)) (justify mirror))
+  )
+  (gr_text PC6 (at 130.25 99.15 180) (layer B.SilkS)
+    (effects (font (size 0.5 0.5) (thickness 0.1)) (justify mirror))
+  )
+  (gr_text "PD2/\nIRQ" (at 137.75 101.35 180) (layer B.SilkS)
+    (effects (font (size 0.5 0.5) (thickness 0.1)) (justify mirror))
+  )
+  (gr_text PD0 (at 130.25 101.7 180) (layer B.SilkS)
+    (effects (font (size 0.5 0.5) (thickness 0.1)) (justify mirror))
+  )
+  (gr_text PB6 (at 137.5 104.1 180) (layer B.SilkS)
+    (effects (font (size 0.5 0.5) (thickness 0.1)) (justify mirror))
+  )
+  (gr_text PD1 (at 130.35 104.2 180) (layer B.SilkS)
+    (effects (font (size 0.5 0.5) (thickness 0.1)) (justify mirror))
+  )
+  (gr_text PD4 (at 137.6 106.7 180) (layer B.SilkS)
+    (effects (font (size 0.5 0.5) (thickness 0.1)) (justify mirror))
+  )
+  (gr_text "PD3/\nRES" (at 130.35 106.45 180) (layer B.SilkS)
+    (effects (font (size 0.5 0.5) (thickness 0.1)) (justify mirror))
+  )
+  (gr_text AERF (at 140 91.55 180) (layer B.SilkS)
+    (effects (font (size 0.5 0.5) (thickness 0.1)) (justify mirror))
+  )
+  (gr_text PB5/SCK (at 148.25 91.55 180) (layer B.SilkS)
+    (effects (font (size 0.5 0.5) (thickness 0.1)) (justify mirror))
+  )
+  (gr_text ADC6 (at 139.9 94.05 180) (layer B.SilkS)
+    (effects (font (size 0.5 0.5) (thickness 0.1)) (justify mirror))
+  )
+  (gr_text VCC (at 147.25 94 180) (layer B.SilkS)
+    (effects (font (size 0.5 0.5) (thickness 0.1)) (justify mirror))
+  )
+  (gr_text GND (at 147.3 96.5 180) (layer B.SilkS)
+    (effects (font (size 0.5 0.5) (thickness 0.1)) (justify mirror))
+  )
+  (gr_text "PB3/\nMOSI" (at 140 96.25 180) (layer B.SilkS)
+    (effects (font (size 0.5 0.5) (thickness 0.1)) (justify mirror))
+  )
+  (gr_text PB4/MISO (at 148.3 99.1 180) (layer B.SilkS)
+    (effects (font (size 0.5 0.5) (thickness 0.1)) (justify mirror))
+  )
+  (gr_text "PB1\n/CE" (at 140.2 98.8 180) (layer B.SilkS)
+    (effects (font (size 0.5 0.5) (thickness 0.1)) (justify mirror))
+  )
+  (gr_text PB2/CSN (at 148.15 101.6 180) (layer B.SilkS)
+    (effects (font (size 0.5 0.5) (thickness 0.1)) (justify mirror))
+  )
+  (gr_text PB0 (at 140.2 101.6 180) (layer B.SilkS)
+    (effects (font (size 0.5 0.5) (thickness 0.1)) (justify mirror))
+  )
+  (gr_text PD7 (at 147.25 104.15 180) (layer B.SilkS)
+    (effects (font (size 0.5 0.5) (thickness 0.1)) (justify mirror))
+  )
+  (gr_text PD6 (at 140.1 104.2 180) (layer B.SilkS)
+    (effects (font (size 0.5 0.5) (thickness 0.1)) (justify mirror))
+  )
+  (gr_text "PD5\n" (at 147.2 106.7 180) (layer B.SilkS)
+    (effects (font (size 0.5 0.5) (thickness 0.1)) (justify mirror))
+  )
+  (gr_text PB7 (at 139.95 106.8 180) (layer B.SilkS)
+    (effects (font (size 0.5 0.5) (thickness 0.1)) (justify mirror))
+  )
   (gr_line (start 129.2 91.1) (end 156.2 91.1) (layer Edge.Cuts) (width 0.05))

Commit message: Add files via upload
Parts:
- added P3: HEADER_1x7, Connector_PinHeader_2.54mm:PinHeader_1x07_P2.54mm_Vertical, B.Cu at (131.4, 92.5)
- P1: value HEADER_2x7 -> HEADER_1x7; footprint Connector_PinHeader_2.54mm:PinHeader_2x07_P2.54mm_Vertical_SMD -> Connector_PinHeader_2.54mm:PinHeader_1x07_P2.54mm_Vertical
- P2: footprint Connector_PinHeader_2.54mm:PinHeader_2x07_P2.54mm_Vertical_SMD -> Connector_PinHeader_2.54mm:PinHeader_2x07_P2.54mm_Vertical
- moved P1 14.4 mm to (131.4, 107.7), turned to 270 degrees
- moved P2 10.9 mm to (126.3, 107.7)
- moved R2 0.38 mm to (133.1, 105.8)
Connections:
- P1 pad 4: Net-(P1-Pad4) -> CE
- P1 pad 6: CSN -> Net-(P1-Pad6)
- P1 pad 7: CE -> MOSI
- U3 pad 10: Net-(P1-Pad3) -> Net-(P1-Pad2)
- U3 pad 11: Net-(P1-Pad4) -> Net-(P1-Pad6)
- U3 pad 12: Net-(P1-Pad5) -> Net-(P1-Pad3)
- U3 pad 19: Net-(P1-Pad11) -> Net-(P3-Pad2)
- U3 pad 20: Net-(P1-Pad13) -> Net-(P3-Pad1)
- U3 pad 9: Net-(P1-Pad2) -> Net-(P1-Pad5)
Routing:
- net 3,3V: track 79.0 -> 54.7 mm, vias 5 -> 4
- net GND: track 78.2 -> 59.4 mm, vias 6 -> 5
- net CE: track 25.4 -> 44.2 mm
- net Net-(P1-Pad4): track 18.3 -> 0.00 mm, vias 1 -> 0
- net MOSI: track 3.63 -> 18.2 mm, vias 1 -> 0
- net CSN: track 34.2 -> 21.4 mm
- net Net-(P1-Pad6): track 0.00 -> 9.88 mm
- net Net-(P2-Pad1): track 4.32 -> 13.4 mm, vias 1 -> 0
- net Net-(P1-Pad3): track 4.64 -> 12.8 mm
- net Net-(P2-Pad12): track 4.85 -> 12.6 mm
- net Net-(P1-Pad11): track 7.69 -> 0.00 mm, vias 1 -> 0
- net Net-(P2-Pad4): track 3.77 -> 11.3 mm
- net Net-(P1-Pad13): track 6.96 -> 0.00 mm, vias 1 -> 0
- net SCK: track 15.8 -> 8.82 mm, vias 1 -> 0
- net Net-(P3-Pad1): track 0.00 -> 6.33 mm
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- added copper zone on F.Cu, net GND
Other:
- board size 27 x 18 mm -> 31 x 18 mm
- board text added: "/PB1"
- board text added: "AREF"
- board text added: "CE"
- board text added: "IRQ"
- board text added: "MISO"
- board text added: "MOSI/PB3"
- board text added: "PB4/"
- board text added: "PD2"
- board text added: "PD3"
- board text added: "VDD"
- board text removed: "AERF"
- board text removed: "PB1 /CE"
- board text removed: "PB3/ MOSI"
- board text removed: "PB4/MISO"
- board text removed: "PD2/ IRQ"
- board text removed: "PD3/ RES"
- board text removed: "VCC"
