File: kicad/MySensors328p.sch (KiCad schematic (older format))
At the start: 22 parts, among them J1 U.FL, J2 U.FL, P1 HEADER_2x7, P2 HEADER_2x7, U1 NRF24L01, U3 ATmega328P-AU, Y1 16 MHz

Commit message: Add files via upload
Parts:
- removed P1: HEADER_2x7, Connector_PinHeader_2.54mm:PinHeader_2x07_P2.54mm_Vertical_SMD, symbol header:HEADER_2x7
- added P1, P3: HEADER_1x7, Connector_PinHeader_2.54mm:PinHeader_1x07_P2.54mm_Vertical, symbol header:HEADER_1x7
- P2: footprint Connector_PinHeader_2.54mm:PinHeader_2x07_P2.54mm_Vertical_SMD -> Connector_PinHeader_2.54mm:PinHeader_2x07_P2.54mm_Vertical
Connections:
- net 3,3V: now also P3.6 (P6)
- net CE: now also P1.4 (P4)
- net CSN: now also P3.3 (P3)
- net GND: now also P3.7 (P7)
- net MISO: now also P3.4 (P4)
- net MOSI: now also P1.7 (P7)
- net SCK: now also P3.5 (P5)
- net at U3.10 (PD6): now also P1.2 (P2)
- net at U3.11 (PD7): now also P1.6 (P6)
- net at U3.12 (PB0): now also P1.3 (P3)
- net at U3.19 (ADC6): now also P3.2 (P2)
- net at U3.20 (AREF): now also P3.1 (P1)
- net at U3.8 (XTAL2/PB7): now also P1.1 (P1)
- net at U3.9 (PD5): now also P1.5 (P5)
Changed lines of the file:
@@
 	2350 4150 2450 4150
-$Comp
-L header:HEADER_2x7 P1
-U 1 1 5B8C3CEA
-P 8900 2750
-F 0 "P1" H 8900 3348 40  0000 C CNN
-F 1 "HEADER_2x7" H 8900 3272 40  0000 C CNN
-F 2 "Connector_PinHeader_2.54mm:PinHeader_2x07_P2.54mm_Vertical_SMD" H 8900 3181 60  0000 C CNN
-F 3 "" H 8900 2750 60  0000 C CNN
-	1    8900 2750
-	1    0    0    -1
-$EndComp
 $Comp
 L MySensors328p-rescue:R-imm_lib-impulse-rescue R2
@@
 3,3V
 Wire Wire Line
-	8750 2450 7800 2450
+	8450 2450 7800 2450
 Wire Wire Line
 	7800 2450 7800 3100
@@
 	7800 3100 6850 3100
 Wire Wire Line
-	8750 2550 7850 2550
+	8450 2550 7850 2550
 Wire Wire Line
 	7850 2550 7850 4700
@@
 	7850 4700 6850 4700
 Wire Wire Line
-	8750 2650 7900 2650
+	8450 2650 7900 2650
 Wire Wire Line
 	7900 2650 7900 2400
@@
 	7900 2400 6850 2400
 Wire Wire Line
-	8750 2750 8000 2750
+	8450 2750 8000 2750
 Wire Wire Line
 	8000 2750 8000 2500
@@
 	8000 2500 6850 2500
 Wire Wire Line
-	8750 2850 7750 2850
-Wire Wire Line
-	7750 2850 7750 2700
-Wire Wire Line
 	7750 2700 6850 2700
 Wire Wire Line
-	8750 2950 8050 2950
-Wire Wire Line
-	8050 2950 8050 2000
-Wire Wire Line
-	8050 2000 5550 2000
-Wire Wire Line
 	5550 2000 5550 2600
 Wire Wire Line
 	5550 2600 5650 2600
 Wire Wire Line
-	8750 3050 8100 3050
-Wire Wire Line
-	8100 3050 8100 1950
-Wire Wire Line
-	8100 1950 5500 1950
-Wire Wire Line
 	5500 1950 5500 2400
 Wire Wire Line
 	5500 2400 5650 2400
 Wire Wire Line
-	9050 2450 9550 2450
-Wire Wire Line
-	9550 2450 9550 3250
-Wire Wire Line
-	9550 3250 7900 3250
-Wire Wire Line
-	7900 3250 7900 4600
-Wire Wire Line
 	7900 4600 6850 4600
 Wire Wire Line
-	9050 2550 9500 2550
-Wire Wire Line
-	9500 2550 9500 3300
-Wire Wire Line
-	9500 3300 7950 3300
-Wire Wire Line
-	7950 3300 7950 4800
-Wire Wire Line
 	7950 4800 6850 4800
 Wire Wire Line
-	9050 2650 9450 2650
+	9100 2650 9450 2650
 Wire Wire Line
 	9450 2650 9450 2300
@@
 	7650 2600 6850 2600
 Wire Wire Line
-	9050 2750 9400 2750
+	9100 2750 9400 2750
 Wire Wire Line
 	9400 2750 9400 2200
@@
 Wire Wire Line
 	7600 2800 6850 2800
-Wire Wire Line
-	9050 2850 9450 2850
 Wire Wire Line
 	9450 2850 9450 5100
@@
 Connection ~ 6250 5100
 Wire Wire Line
-	9050 2950 9350 2950
+	9100 2950 9350 2950
 Wire Wire Line
 	9350 2950 9350 2100
@@
 	9350 2100 6350 2100
 Connection ~ 6350 2100
-Wire Wire Line
-	9050 3050 9100 3050
-Wire Wire Line
-	9100 3050 9100 3200
-Wire Wire Line
-	9100 3200 7650 3200
 Wire Wire Line
 	7650 3200 7650 2900
@@
 F 0 "P2" H 8900 4848 40  0000 C CNN
 F 1 "HEADER_2x7" H 8900 4772 40  0000 C CNN
-F 2 "Connector_PinHeader_2.54mm:PinHeader_2x07_P2.54mm_Vertical_SMD" H 8900 4681 60  0000 C CNN
+F 2 "Connector_PinHeader_2.54mm:PinHeader_2x07_P2.54mm_Vertical" H 8900 4681 60  0000 C CNN
 F 3 "" H 8900 4250 60  0000 C CNN
 	1    8900 4250
@@
 Wire Wire Line
 	4150 3550 4150 3950
+$Comp
+L header:HEADER_1x7 P1
+U 1 1 5B8DB30F
+P 8600 2750
+F 0 "P1" H 8678 2841 40  0000 L CNN
+F 1 "HEADER_1x7" H 8678 2765 40  0000 L CNN
+F 2 "Connector_PinHeader_2.54mm:PinHeader_1x07_P2.54mm_Vertical" H 8678 2674 60  0000 L CNN
+F 3 "" H 8600 2750 60  0000 C CNN
+	1    8600 2750
+	1    0    0    -1
+$EndComp
+$Comp
+L header:HEADER_1x7 P3
+U 1 1 5B8DB385
+P 8950 2750
+F 0 "P3" H 8894 3348 40  0000 C CNN
+F 1 "HEADER_1x7" H 8894 3272 40  0000 C CNN
+F 2 "Connector_PinHeader_2.54mm:PinHeader_1x07_P2.54mm_Vertical" H 8894 3181 60  0000 C CNN
+F 3 "" H 8950 2750 60  0000 C CNN
+	1    8950 2750
+	-1   0    0    -1
+$EndComp
+Wire Wire Line
+	9500 1950 9500 2450
+Wire Wire Line
+	9500 2450 9100 2450
+Wire Wire Line
+	5500 1950 9500 1950
+Wire Wire Line
+	7950 2950 8450 2950
+Wire Wire Line
+	7950 2950 7950 4800
+Wire Wire Line
+	9300 2000 9300 2550
+Wire Wire Line
+	9300 2550 9100 2550
+Wire Wire Line
+	5550 2000 9300 2000
+Wire Wire Line
+	7900 2850 8450 2850
+Wire Wire Line
+	7900 2850 7900 4600
+Wire Wire Line
+	7750 3050 8450 3050
+Wire Wire Line
+	7750 2700 7750 3050
+Wire Wire Line
+	9250 3200 9250 2850
+Wire Wire Line
+	9250 2850 9100 2850
+Wire Wire Line
+	7650 3200 9250 3200
+Wire Wire Line
+	9450 2850 9600 2850
+Wire Wire Line
+	9600 2850 9600 3050
+Wire Wire Line
+	9600 3050 9100 3050
 $EndSCHEMATC
